File: NumPad.sch (KiCad schematic (older format))
At the start: 56 parts, among them J1 USB_B_Micro, K1 numlk, K2 /, K3 *, K4 -, SW1 RESET, U1 ATmega32U4RC-AU, X1 18pF

Commit message: Esquemático terminado y PCB empezada
Parts:
- removed D? (x3): D_ALT, symbol Device:D_ALT
- removed K? (x2): -, symbol keyboard_parts:KEYSW
- removed K?: *, symbol keyboard_parts:KEYSW
- C1, C2, C3, C4, C5, C6, C7, C8: footprint (none) -> Capacitor_SMD:C_0805_2012Metric
- D1, D2, D3, D4: footprint (none) -> Diode_SMD:D_SOD-123
- D10, D11, D12, D13, D14, D15, D16, D17, D5, D6, D7, D8, D9: renamed from D?; footprint (none) -> Diode_SMD:D_SOD-123
- J1: footprint (none) -> keyboard_parts:USB_microB
- K1, K2, K3, K4: footprint (none) -> Button_Switch_Keyboard:SW_Cherry_MX_1.00u_PCB
- K10: renamed from K?; value / -> 5; footprint (none) -> Button_Switch_Keyboard:SW_Cherry_MX_1.00u_PCB
- K11: renamed from K?; value * -> 6; footprint (none) -> Button_Switch_Keyboard:SW_Cherry_MX_1.00u_PCB
- K12: renamed from K?; value - -> enter; footprint (none) -> Button_Switch_Keyboard:SW_Cherry_MX_2.00u_Vertical_PCB
- K13: renamed from K?; value numlk -> 1; footprint (none) -> Button_Switch_Keyboard:SW_Cherry_MX_1.00u_PCB
- K14: renamed from K?; value / -> 2; footprint (none) -> Button_Switch_Keyboard:SW_Cherry_MX_1.00u_PCB
- K15: renamed from K?; value * -> 3; footprint (none) -> Button_Switch_Keyboard:SW_Cherry_MX_1.00u_PCB
- K16: renamed from K?; value numlk -> 0; footprint (none) -> Button_Switch_Keyboard:SW_Cherry_MX_2.00u_PCB
- K17: renamed from K?; value / -> .; footprint (none) -> Button_Switch_Keyboard:SW_Cherry_MX_1.00u_PCB
- K5: renamed from K?; value numlk -> 7; footprint (none) -> Button_Switch_Keyboard:SW_Cherry_MX_1.00u_PCB
- K6: renamed from K?; value / -> 8; footprint (none) -> Button_Switch_Keyboard:SW_Cherry_MX_1.00u_PCB
- K7: renamed from K?; value * -> 9; footprint (none) -> Button_Switch_Keyboard:SW_Cherry_MX_1.00u_PCB
- K8: renamed from K?; value - -> +; footprint (none) -> Button_Switch_Keyboard:SW_Cherry_MX_2.00u_Vertical_PCB
- K9: renamed from K?; value numlk -> 4; footprint (none) -> Button_Switch_Keyboard:SW_Cherry_MX_1.00u_PCB
- R1, R2: footprint (none) -> Resistor_SMD:R_0805_2012Metric
- R3, R4: footprint (none) -> Resistor_SMD:R_0603_1608Metric
- SW1: footprint (none) -> Button_Switch_THT:SW_PUSH_6mm
- X1: footprint (none) -> Crystal:Crystal_SMD_SeikoEpson_FA238-4Pin_3.2x2.5mm
Connections:
- net labels added: col1, col2, col3, col4, row2, row3, row4, row5
- wire segments 184 -> 194
- no-connect marks 0 -> 16
Other:
- moved on the sheet: D17, K17
